File: Modified designs/Electronics/hot-end-connector/hot-end-connector.kicad_pcb (KiCad board)
At the start: 2 copper layers, 34 x 27 mm, 4 parts, among them J1 Conn_01x08_Pin, J2 Conn_01x08_Pin

Commit message: Final (?) PCB design.
Parts:
- added 1N4148: 1N4148, Diode_SMD:D_0805_2012Metric, F.Cu at (45.0, 169.6)
- added D1: LED, LED_SMD:LED_0805_2012Metric, F.Cu at (49.0, 177.0)
- added D2: LED, LED_SMD:LED_0805_2012Metric, F.Cu at (49.0, 170.5)
- added R1: 820R, Resistor_SMD:R_0805_2012Metric, F.Cu at (55.1, 177.0)
- added R2: 220R, Resistor_SMD:R_0805_2012Metric, F.Cu at (49.0, 168.0)
- J1: value Conn_01x08_Pin -> ~; footprint Connector_PinHeader_2.54mm:PinHeader_1x08_P2.54mm_Horizontal -> Connector_PinHeader_2.54mm:PinHeader_1x07_P2.54mm_Horizontal
- J2: value Conn_01x08_Pin -> ~; footprint Connector_PinHeader_2.54mm:PinHeader_1x08_P2.54mm_Horizontal -> Connector_PinHeader_2.54mm:PinHeader_1x08_P2.54mm_Vertical
- moved J1 33.2 mm to (59.0, 160.3), turned to 0 degrees
- moved J2 32.7 mm to (31.0, 176.6), turned to 180 degrees
Connections:
- J1 pad 1: Net-(J1-Pin_1) -> /T-b
- J1 pad 2: Net-(J1-Pin_2) -> /T-a
- J1 pad 3: Net-(J1-Pin_3) -> /probe
- J1 pad 4: Net-(J1-Pin_4) -> /+3V3
- J1 pad 5: Net-(J1-Pin_5) -> /GND
- J1 pad 6: Net-(J1-Pin_6) -> /H-
- J1 pad 7: Net-(J1-Pin_7) -> /+12V
- J2 pad 1: Net-(J1-Pin_8) -> /+12V
- J2 pad 2: Net-(J1-Pin_7) -> /H-
- J2 pad 3: Net-(J1-Pin_6) -> /GND
- J2 pad 4: Net-(J1-Pin_5) -> /probe
- J2 pad 5: Net-(J1-Pin_4) -> /T-a
- J2 pad 6: Net-(J1-Pin_3) -> /T-b
- J2 pad 7: Net-(J1-Pin_2) -> /GND
- J2 pad 8: Net-(J1-Pin_1) -> /+12V
Routing:
- net /+12V: track 0.00 -> 56.2 mm
- net /GND: track 0.00 -> 51.6 mm
- net /probe: track 0.00 -> 35.9 mm, vias 0 -> 1
- net Net-(J1-Pin_5): track 34.2 -> 0.00 mm
- net /H-: track 0.00 -> 33.8 mm, vias 0 -> 1
- net Net-(J1-Pin_1): track 30.8 -> 0.00 mm
- net Net-(J1-Pin_8): track 30.5 -> 0.00 mm
- net Net-(J1-Pin_7): track 30.1 -> 0.00 mm
- net Net-(J1-Pin_2): track 29.9 -> 0.00 mm
- net Net-(J1-Pin_6): track 29.6 -> 0.00 mm
- net /T-b: track 0.00 -> 29.5 mm
- net /T-a: track 0.00 -> 29.5 mm
- net Net-(J1-Pin_3): track 29.0 -> 0.00 mm
- net Net-(J1-Pin_4): track 28.4 -> 0.00 mm
- net /+3V3: track 0.00 -> 9.14 mm
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- added copper zone on B.Cu, net /GND
- added copper zone on F.Cu, net /GND
Other:
- board text added: "F+"
- board text added: "F-"
- board text added: "H"
- board text added: "H+"
- board text added: "H-"
- board text added: "P"
- board text added: "P3v3"
- board text added: "Pg"
- board text added: "RepRap Ltd https://reprapltd.com Hot End Connector Licence: GPL"
- board text added: "T"
- board text added: "heat"
- board text added: "touch"
